File: mainboard_2024_a.kicad_pcb (KiCad board)
At the start: 2 copper layers, 8 parts, among them J1 Raspberry_Pi_2_3, M1 Conn_01x03_Socket, M2 Conn_01x03_Socket, M3 Conn_01x03_Socket, M4 Conn_01x03_Socket, M5 Conn_01x03_Socket

Commit message: add text
Other:
- board text added: "5V"
- board text added: "GND"
- board text added: "dir"
- board text added: "pwm"
Changed lines of the file:
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@@
 		)
 		(property "Value" "Conn_01x03_Socket"
-			(at 1.016 -10.795 180)
+			(at 0.381 -24.003 180)
 			(layer "F.Fab")
 			(effects
@@
 		)
 	)
+	(gr_text "dir"
+		(at 122.555 115.57 0)
+		(layer "B.Cu")
+		(effects
+			(font
+				(size 1 1)
+				(thickness 0.1)
+			)
+			(justify left bottom)
+		)
+	)
+	(gr_text "5V"
+		(at 113.03 75.438 0)
+		(layer "B.Cu")
+		(effects
+			(font
+				(size 1 1)
+				(thickness 0.1)
+			)
+			(justify left bottom)
+		)
+	)
+	(gr_text "pwm\n"
+		(at 122.555 112.649 0)
+		(layer "B.Cu")
+		(effects
+			(font
+				(size 1 1)
+				(thickness 0.1)
+			)
+			(justify left bottom)
+		)
+	)
+	(gr_text "GND"
+		(at 115.824 75.311 0)
+		(layer "B.Cu")
+		(effects
+			(font
+				(size 1 1)
+				(thickness 0.1)
+			)
+			(justify left bottom)
+		)
+	)
+	(gr_text "GND\n"
+		(at 122.428 110.236 0)
+		(layer "B.Cu")
+		(effects
+			(font
+				(size 1 1)
+				(thickness 0.1)
+			)
+			(justify left bottom)
+		)
+	)

Commit message: ロボコン辞めます
Parts:
- moved fun1 0.09 mm to (124.5, 78.8)
Routing:
- net Net-(M1-Pin_1): track 85.9 -> 102.6 mm
- net Net-(fun1-Pin_1): track 21.9 -> 28.0 mm
- net Net-(J1-PWM0/GPIO12): track 34.4 -> 30.5 mm
- net Net-(J1-GPIO25): track 24.7 -> 25.7 mm
Other:
- board text added: "1"
- board text added: "2"
- board text added: "3"
- board text added: "4"
- board text added: "5"

Commit message: update
Parts:
- added C1: 100u, Capacitor_SMD:C_1206_3216Metric_Pad1.33x1.80mm_HandSolder, F.Cu at (161.4, 85.0)
- added M6: Conn_01x03_Socket, Connector_JST:JST_XH_B3B-XH-A_1x03_P2.50mm_Vertical, F.Cu at (145.6, 111.4)
- J1: moved to B.Cu
- M1, M2, M3, M4, M5: footprint Connector_JST:JST_PH_B3B-PH-K_1x03_P2.00mm_Vertical -> Connector_JST:JST_XH_B3B-XH-A_1x03_P2.50mm_Vertical
- fun1, power1: footprint Connector_JST:JST_PH_B2B-PH-K_1x02_P2.00mm_Vertical -> Connector_JST:JST_XH_B2B-XH-A_1x02_P2.50mm_Vertical
- moved J1 59.3 mm to (166.0, 78.1), turned to 180 degrees
- moved power1 44.3 mm to (158.6, 80.2), turned to 180 degrees
- moved M1 38.9 mm to (155.8, 88.1)
- moved M3 38.9 mm to (155.8, 99.7)
- moved M5 38.9 mm to (155.8, 111.4)
- moved fun1 24.9 mm to (149.3, 80.3), turned to 180 degrees
- moved M2 18.6 mm to (145.6, 88.1)
- moved M4 18.6 mm to (145.6, 99.7)
Connections:
- net Net-(M1-Pin_1) renamed GND
- net Net-(fun1-Pin_1) renamed VCC
- J1 pad 3: unconnected-(J1-SDA/GPIO2-Pad3) -> Net-(J1-SDA/GPIO2)
- J1 pad 33: unconnected-(J1-PWM1/GPIO13-Pad33) -> Net-(J1-PWM1/GPIO13)
Routing:
- net Net-(J1-SDA/GPIO2): track 0.00 -> 74.7 mm, vias 0 -> 1
- net Net-(J1-PWM1/GPIO13): track 0.00 -> 32.0 mm, vias 0 -> 1
- net GND: track 102.6 -> 117.6 mm
- net VCC: track 28.0 -> 36.6 mm
- net Net-(J1-GPIO17): track 10.9 -> 17.7 mm
- net Net-(J1-GPIO18/PWM0): track 13.2 -> 17.9 mm
- net Net-(J1-GPIO16): track 17.0 -> 18.2 mm
- net Net-(J1-GPIO27): track 22.6 -> 23.6 mm
- net Net-(J1-GPIO25): track 25.7 -> 26.5 mm
- net Net-(J1-GPIO24): track 14.8 -> 15.4 mm
- added copper zone on B.Cu, net GND
- added copper zone on F.Cu, net GND
Other:
- board outline added: 30 x 64.2 mm
- board text added: "PWM"
- board text removed: "pwm"

Commit message: add 7 8 9
Parts:
- added M7: Conn_01x03_Socket, Connector_JST:JST_XH_B3B-XH-A_1x03_P2.50mm_Vertical, F.Cu at (134.6, 87.8)
- added M8: Conn_01x03_Socket, Connector_JST:JST_XH_B3B-XH-A_1x03_P2.50mm_Vertical, F.Cu at (134.6, 99.6)
- added M9: Conn_01x03_Socket, Connector_JST:JST_XH_B3B-XH-A_1x03_P2.50mm_Vertical, F.Cu at (134.6, 111.4)
Connections:
- J1 pad 19: unconnected-(J1-MOSI0/GPIO10-Pad19) -> Net-(J1-MOSI0/GPIO10)
- J1 pad 21: unconnected-(J1-MISO0/GPIO9-Pad21) -> Net-(J1-MISO0/GPIO9)
- J1 pad 23: unconnected-(J1-SCLK0/GPIO11-Pad23) -> Net-(J1-SCLK0/GPIO11)
- J1 pad 24: unconnected-(J1-~{CE0}/GPIO8-Pad24) -> Net-(J1-~{CE0}/GPIO8)
- J1 pad 5: unconnected-(J1-SCL/GPIO3-Pad5) -> Net-(J1-SCL/GPIO3)
- J1 pad 7: unconnected-(J1-GCLK0/GPIO4-Pad7) -> Net-(J1-GCLK0/GPIO4)
Routing:
- net GND: track 117.6 -> 243.2 mm, vias 1 -> 2
- net Net-(J1-~{CE0}/GPIO8): track 0.00 -> 49.6 mm, vias 0 -> 1
- net Net-(J1-GCLK0/GPIO4): track 0.00 -> 41.7 mm, vias 0 -> 1
- net Net-(J1-MOSI0/GPIO10): track 0.00 -> 35.2 mm, vias 0 -> 1
- net Net-(J1-SCL/GPIO3): track 0.00 -> 35.1 mm, vias 0 -> 1
- net Net-(J1-SCLK0/GPIO11): track 0.00 -> 34.6 mm, vias 0 -> 1
Other:
- board size 30 x 64.2 mm -> 45.6 x 64.2 mm
