File: mainboard_2024_a.kicad_sch (KiCad schematic)
At the start: 8 parts, among them J1 Raspberry_Pi_2_3, M1 Conn_01x03_Socket, M2 Conn_01x03_Socket, M3 Conn_01x03_Socket, M4 Conn_01x03_Socket, M5 Conn_01x03_Socket

Commit message: ロボコン辞めます
Connections:
- net GND: no longer names the net of J1.14 (GND), J1.20 (GND), J1.25 (GND), J1.30 (GND), J1.34 (GND), J1.39 (GND), J1.6 (GND), J1.9 (GND), M1.1 (Pin_1), M2.1 (Pin_1), M3.1 (Pin_1), M4.1 (Pin_1), M5.1 (Pin_1), fun1.2 (Pin_2), power1.2 (Pin_2)
- net VCC: no longer names the net of J1.2 (5V), J1.4 (5V), fun1.1 (Pin_1), power1.1 (Pin_1)
Changed lines of the file:
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@@
-	)
-	(junction
-		(at 200.66 30.48)
-		(diameter 0)
-		(color 0 0 0 0)
-	)
-	(junction
-		(at 187.96 30.48)
-		(diameter 0)
-		(color 0 0 0 0)
-	)
-	(junction
-		(at 205.74 97.79)
-		(diameter 0)
-		(color 0 0 0 0)
 	)
 	(junction
@@
 	(wire
 		(pts
-			(xy 200.66 30.48) (xy 226.06 30.48)
-		)
-		(stroke
-			(width 0)
-			(type default)
-		)
-	)
-	(wire
-		(pts
 			(xy 166.37 87.63) (xy 166.37 97.79)
 		)
@@
 	(wire
 		(pts
-			(xy 166.37 30.48) (xy 187.96 30.48)
-		)
-		(stroke
-			(width 0)
-			(type default)
-		)
-	)
-	(wire
-		(pts
-			(xy 205.74 97.79) (xy 231.14 97.79)
+			(xy 166.37 30.48) (xy 226.06 30.48)
+		)
+		(stroke
+			(width 0)
+			(type default)
+		)
+	)
+	(wire
+		(pts
+			(xy 168.91 97.79) (xy 231.14 97.79)
 		)
 		(stroke
@@
 	(wire
 		(pts
-			(xy 168.91 97.79) (xy 205.74 97.79)
-		)
-		(stroke
-			(width 0)
-			(type default)
-		)
-	)
-	(wire
-		(pts
 			(xy 201.93 44.45) (xy 201.93 49.53)
 		)
@@
 		(pts
 			(xy 172.72 102.87) (xy 142.24 102.87)
-		)
-		(stroke
-			(width 0)
-			(type default)
-		)
-	)
-	(wire
-		(pts
-			(xy 187.96 30.48) (xy 200.66 30.48)
 		)
 		(stroke
@@
 	)
 	(symbol
-		(lib_id "power:PWR_FLAG")
-		(at 187.96 30.48 0)
-		(unit 1)
-		(exclude_from_sim no)
-		(in_bom yes)
-		(on_board yes)
-		(dnp no)
-		(fields_autoplaced yes)
-		(property "Reference" "#FLG01"
-			(at 187.96 28.575 0)
-			(effects
-				(font
-					(size 1.27 1.27)
-				)
-				(hide yes)
-			)
-		)
-		(property "Value" "PWR_FLAG"
-			(at 187.96 25.4 0)
-			(effects
-				(font
-					(size 1.27 1.27)
-				)
-			)
-		)
-		(property "Footprint" ""
-			(at 187.96 30.48 0)
-			(effects
-				(font
-					(size 1.27 1.27)
-				)
-				(hide yes)
-			)
-		)
-		(property "Datasheet" "~"
-			(at 187.96 30.48 0)
-			(effects
-				(font
-					(size 1.27 1.27)
-				)
-				(hide yes)
-			)
-		)
-		(property "Description" "Special symbol for telling ERC where power comes from"
-			(at 187.96 30.48 0)
-			(effects
-				(font
-					(size 1.27 1.27)
-				)
-				(hide yes)
-			)
-		)
-		(pin "1"
-		)
-		(instances
-			(project ""
-				(path "/c99ec100-acb9-41b5-a70a-0fc7e5a0f69c"
-					(reference "#FLG01")
-					(unit 1)
-				)
-			)
-		)
-	)
-	(symbol
 		(lib_id "Connector:Conn_01x03_Socket")
 		(at 135.89 95.25 180)
@@
 				(path "/c99ec100-acb9-41b5-a70a-0fc7e5a0f69c"
 					(reference "M4")
-					(unit 1)
-				)
-			)
-		)
-	)
-	(symbol
-		(lib_id "power:GND")
-		(at 205.74 97.79 0)
-		(unit 1)
-		(exclude_from_sim no)
-		(in_bom yes)
-		(on_board yes)
-		(dnp no)
-		(fields_autoplaced yes)
-		(property "Reference" "#PWR01"
-			(at 205.74 104.14 0)
-			(effects
-				(font
-					(size 1.27 1.27)
-				)
-				(hide yes)
-			)
-		)
-		(property "Value" "GND"
-			(at 205.74 102.87 0)
-			(effects
-				(font
-					(size 1.27 1.27)
-				)
-			)
-		)
-		(property "Footprint" ""
-			(at 205.74 97.79 0)
-			(effects
-				(font
-					(size 1.27 1.27)
-				)
-				(hide yes)
-			)
-		)
-		(property "Datasheet" ""
-			(at 205.74 97.79 0)
-			(effects
-				(font
-					(size 1.27 1.27)
-				)
-				(hide yes)
-			)
-		)
-		(property "Description" "Power symbol creates a global label with name \"GND\" , ground"
-			(at 205.74 97.79 0)
-			(effects
-				(font
-					(size 1.27 1.27)
-				)
-				(hide yes)
-			)
-		)
-		(pin "1"
-		)
-		(instances
-			(project ""
-				(path "/c99ec100-acb9-41b5-a70a-0fc7e5a0f69c"
-					(reference "#PWR01")
 					(unit 1)
 				)
@@
 					(unit 1)
 				)
-			)
-		)
-	)
-	(symbol
-		(lib_id "power:VCC")
-		(at 200.66 30.48 0)
-		(unit 1)
-		(exclude_from_sim no)
-		(in_bom yes)
-		(on_board yes)
-		(dnp no)
-		(fields_autoplaced yes)
-		(property "Reference" "#PWR02"
-			(at 200.66 34.29 0)
-			(effects
-				(font
-					(size 1.27 1.27)
-				)
-				(hide yes)
-			)
-		)
-		(property "Value" "VCC"
-			(at 200.66 25.4 0)
-			(effects
-				(font
-					(size 1.27 1.27)
-				)
-			)
-		)
-		(property "Footprint" ""
-			(at 200.66 30.48 0)
-			(effects
-				(font
-					(size 1.27 1.27)
-				)
-				(hide yes)
-			)
-		)
-		(property "Datasheet" ""
-			(at 200.66 30.48 0)
-			(effects
-				(font
-					(size 1.27 1.27)
-				)
-				(hide yes)
-			)
-		)
-		(property "Description" "Power symbol creates a global label with name \"VCC\""
-			(at 200.66 30.48 0)
-			(effects
-				(font
-					(size 1.27 1.27)
-				)
-				(hide yes)
-			)
-		)
-		(pin "1"
-		)
-		(instances
-			(project ""
-				(path "/c99ec100-acb9-41b5-a70a-0fc7e5a0f69c"
-					(reference "#PWR02")
-					(unit 1)
-				)

Commit message: update
Parts:
- added C1: 100u, Capacitor_SMD:C_1206_3216Metric_Pad1.33x1.80mm_HandSolder, symbol Device:C
- added M6: Conn_01x03_Socket, Connector_JST:JST_XH_B3B-XH-A_1x03_P2.50mm_Vertical, symbol Connector:Conn_01x03_Socket
- M1, M2, M3, M4, M5: footprint Connector_JST:JST_PH_B3B-PH-K_1x03_P2.00mm_Vertical -> Connector_JST:JST_XH_B3B-XH-A_1x03_P2.50mm_Vertical
- fun1, power1: footprint Connector_JST:JST_PH_B2B-PH-K_1x02_P2.00mm_Vertical -> Connector_JST:JST_XH_B2B-XH-A_1x02_P2.50mm_Vertical
Connections:
- net GND: now reaches J1.14 (GND), J1.20 (GND), J1.25 (GND), J1.30 (GND), J1.34 (GND), J1.39 (GND), J1.6 (GND), J1.9 (GND), M1.1 (Pin_1), M2.1 (Pin_1), M3.1 (Pin_1), M4.1 (Pin_1), M5.1 (Pin_1), fun1.2 (Pin_2), power1.2 (Pin_2)
- net GND: now also C1.2, M6.1 (Pin_1)
- net VCC: now reaches J1.2 (5V), J1.4 (5V), fun1.1 (Pin_1), power1.1 (Pin_1)
- net VCC: now also C1.1
- net at J1.3 (SDA/GPIO2): now also M6.3 (Pin_3)
- net at J1.33 (PWM1/GPIO13): now also M6.2 (Pin_2)

Commit message: add 7 8 9
Parts:
- added M7, M8, M9: Conn_01x03_Socket, Connector_JST:JST_XH_B3B-XH-A_1x03_P2.50mm_Vertical, symbol Connector:Conn_01x03_Socket
Connections:
- net GND: now also M7.1 (Pin_1), M8.1 (Pin_1), M9.1 (Pin_1)
- net at J1.19 (MOSI0/GPIO10): now also M8.2 (Pin_2)
- net at J1.21 (MISO0/GPIO9): now also M8.3 (Pin_3)
- net at J1.23 (SCLK0/GPIO11): now also M9.2 (Pin_2)
- net at J1.24 (~{CE0}/GPIO8): now also M9.3 (Pin_3)
- net at J1.5 (SCL/GPIO3): now also M7.2 (Pin_2)
- net at J1.7 (GCLK0/GPIO4): now also M7.3 (Pin_3)
Other:
- moved on the sheet: C1, J1, M1, M2, M3, M4, M5, M6, fun1, power1
